File: LCC-PNET-Router.kicad_pcb (KiCad board)
At the start: 2 copper layers, 2 parts, among them P1 POCKETBEAGLE-P1, P2 POCKETBEAGLE-P2

Commit message: Start on PCB layout.
Parts:
- added C201: .1 uf, Capacitors_THT:C_Rect_L4.0mm_W2.5mm_P2.50mm, F.Cu at (130.8, 73.7)
- added C202: 47 nf, Capacitors_THT:C_Rect_L4.0mm_W2.5mm_P2.50mm, F.Cu at (146.1, 49.5)
- added C203: 15 uf 15V, Capacitors_THT:CP_Radial_D6.3mm_P2.50mm, F.Cu at (124.5, 73.7)
- added C301: .1 uf, Capacitors_THT:C_Rect_L4.0mm_W2.5mm_P2.50mm, F.Cu at (129.5, 134.6)
- added C302: 47 nf, Capacitors_THT:C_Rect_L4.0mm_W2.5mm_P2.50mm, F.Cu at (147.4, 152.4)
- added C303: 15 uf 15V, Capacitors_THT:CP_Radial_D6.3mm_P2.50mm, F.Cu at (123.2, 134.6)
- added C401: 220 uf 25V, Capacitors_THT:CP_Radial_D8.0mm_P3.50mm, F.Cu at (165.1, 119.4)
- added C402: 22 uf 100V, Capacitors_THT:CP_Radial_D8.0mm_P3.50mm, F.Cu at (173.0, 77.5)
- added D201: CAN Tx, LEDs:LED_D3.0mm, F.Cu at (161.3, 73.7)
- added D202: CAN Rx, LEDs:LED_D3.0mm, F.Cu at (161.3, 77.5)
- added D203: SB240, Diodes_THT:D_DO-15_P10.16mm_Horizontal, F.Cu at (119.4, 52.1)
- added D204: SB240, Diodes_THT:D_DO-15_P10.16mm_Horizontal, F.Cu at (152.4, 50.8)
- added D301: CAN Tx, LEDs:LED_D3.0mm, F.Cu at (162.6, 130.8)
- added D302: CAN Rx, LEDs:LED_D3.0mm, F.Cu at (162.6, 135.9)
- added D401: SB160-E3/54, Diodes_THT:D_DO-41_SOD81_P7.62mm_Horizontal, F.Cu at (172.7, 86.4)
- added J101: USB_A, USB-A-Upright:USB-A-UPRIGHT, F.Cu at (120.6, 88.7)
- added J201: Termination, Pin_Headers:Pin_Header_Straight_2x02_Pitch2.54mm, F.Cu at (139.7, 49.5)
- added J202: RJ45, RJ45-8N-S:RJ45_8N-S, F.Cu at (163.8, 62.9)
- added J203: RJ45, RJ45-8N-S:RJ45_8N-S, F.Cu at (118.6, 63.0)
- added J301: Termination, Pin_Headers:Pin_Header_Straight_2x02_Pitch2.54mm, F.Cu at (141.0, 152.4)
- added J302: PNET, Connectors:RJ12_E, F.Cu at (160.3, 145.3)
- added J303: PNET, Connectors:RJ12_E, F.Cu at (115.8, 145.3)
- added L401: 330 uh, PELowProfile:PE-LowProfile, F.Cu at (167.6, 104.1)
- added R201: 160 Ohms, Resistors_THT:R_Axial_DIN0204_L3.6mm_D1.6mm_P1.90mm_Vertical, F.Cu at (156.8, 73.7)
- added R202: 160 Ohms, Resistors_THT:R_Axial_DIN0204_L3.6mm_D1.6mm_P1.90mm_Vertical, F.Cu at (156.8, 77.5)
- added R203: 60 Ohms, Resistors_THT:R_Axial_DIN0204_L3.6mm_D1.6mm_P2.54mm_Vertical, F.Cu at (133.3, 49.5)
- added R204: 60 Ohms, Resistors_THT:R_Axial_DIN0204_L3.6mm_D1.6mm_P2.54mm_Vertical, F.Cu at (133.3, 47.0)
- added R301: 160 Ohms, Resistors_THT:R_Axial_DIN0204_L3.6mm_D1.6mm_P1.90mm_Vertical, F.Cu at (158.1, 130.8)
- added R302: 160 Ohms, Resistors_THT:R_Axial_DIN0204_L3.6mm_D1.6mm_P1.90mm_Vertical, F.Cu at (158.1, 134.6)
- added R303: 60 Ohms, Resistors_THT:R_Axial_DIN0204_L3.6mm_D1.6mm_P2.54mm_Vertical, F.Cu at (134.6, 152.4)
- added R304: 60 Ohms, Resistors_THT:R_Axial_DIN0204_L3.6mm_D1.6mm_P2.54mm_Vertical, F.Cu at (134.6, 148.6)
- added T201: LCC Power Out, Connectors_Terminal_Blocks:TerminalBlock_Pheonix_MPT-2.54mm_2pol, F.Cu at (118.1, 44.5)
- added T202: LCC Power In, Connectors_Terminal_Blocks:TerminalBlock_Pheonix_MPT-2.54mm_2pol, F.Cu at (162.6, 43.2)
- added U201: LM358, Housings_DIP:DIP-8_W7.62mm, F.Cu at (149.9, 71.1)
- added U202: TCAN332DR, Housings_SOIC:SOIC-8-1EP_3.9x4.9mm_Pitch1.27mm, F.Cu at (136.5, 75.1)
- added U301: LM358, Housings_DIP:DIP-8_W7.62mm, F.Cu at (142.2, 137.2)
- added U302: TCAN332DR, Housings_SOIC:SOIC-8-1EP_3.9x4.9mm_Pitch1.27mm, F.Cu at (136.5, 133.2)
- added U401: LM2574N-5.0, Housings_DIP:DIP-8_W7.62mm, F.Cu at (161.3, 83.8)
Connections:
- P1 pad 1: (no net) -> +5V
- P1 pad 10: (no net) -> Net-(P1-Pad10)
- P1 pad 11: (no net) -> Net-(J101-Pad3)
- P1 pad 12: (no net) -> Net-(P1-Pad12)
- P1 pad 13: (no net) -> GND
- P1 pad 14: (no net) -> +3V3
- P1 pad 15: (no net) -> GND
- P1 pad 16: (no net) -> GND
- P1 pad 17: (no net) -> Net-(P1-Pad17)
- P1 pad 18: (no net) -> Net-(P1-Pad18)
- P1 pad 19: (no net) -> Net-(P1-Pad19)
- P1 pad 2: (no net) -> Net-(P1-Pad2)
- P1 pad 20: (no net) -> Net-(P1-Pad20)
- P1 pad 21: (no net) -> Net-(P1-Pad21)
- P1 pad 22: (no net) -> GND
- P1 pad 23: (no net) -> Net-(P1-Pad23)
- P1 pad 24: (no net) -> Net-(P1-Pad24)
- P1 pad 25: (no net) -> Net-(P1-Pad25)
- P1 pad 26: (no net) -> /CAN0_TX
- P1 pad 27: (no net) -> Net-(P1-Pad27)
- P1 pad 28: (no net) -> /CAN0_RX
- P1 pad 29: (no net) -> Net-(P1-Pad29)
- P1 pad 3: (no net) -> Net-(P1-Pad3)
- P1 pad 30: (no net) -> Net-(P1-Pad30)
- P1 pad 31: (no net) -> Net-(P1-Pad31)
- P1 pad 32: (no net) -> Net-(P1-Pad32)
- P1 pad 33: (no net) -> Net-(P1-Pad33)
- P1 pad 34: (no net) -> Net-(P1-Pad34)
- P1 pad 35: (no net) -> Net-(P1-Pad35)
- P1 pad 36: (no net) -> Net-(P1-Pad36)
- P1 pad 4: (no net) -> Net-(P1-Pad4)
- P1 pad 5: (no net) -> +5V
- P1 pad 6: (no net) -> Net-(P1-Pad6)
- P1 pad 7: (no net) -> Net-(P1-Pad7)
- P1 pad 8: (no net) -> Net-(P1-Pad8)
- P1 pad 9: (no net) -> Net-(J101-Pad2)
- P2 pad 1: (no net) -> Net-(P2-Pad1)
- P2 pad 10: (no net) -> Net-(P2-Pad10)
- P2 pad 11: (no net) -> /CAN1_TX
- P2 pad 12: (no net) -> Net-(P2-Pad12)
- P2 pad 13: (no net) -> Net-(P2-Pad13)
- P2 pad 14: (no net) -> Net-(P2-Pad14)
- P2 pad 15: (no net) -> GND
- P2 pad 16: (no net) -> Net-(P2-Pad16)
- P2 pad 17: (no net) -> Net-(P2-Pad17)
- P2 pad 18: (no net) -> Net-(P2-Pad18)
- P2 pad 19: (no net) -> Net-(P2-Pad19)
- P2 pad 2: (no net) -> Net-(P2-Pad2)
- P2 pad 20: (no net) -> Net-(P2-Pad20)
- P2 pad 21: (no net) -> GND
- P2 pad 22: (no net) -> Net-(P2-Pad22)
- P2 pad 23: (no net) -> +3V3
- P2 pad 24: (no net) -> Net-(P2-Pad24)
- P2 pad 25: (no net) -> Net-(P2-Pad25)
- P2 pad 26: (no net) -> Net-(P2-Pad26)
- P2 pad 27: (no net) -> Net-(P2-Pad27)
- P2 pad 28: (no net) -> Net-(P2-Pad28)
- P2 pad 29: (no net) -> Net-(P2-Pad29)
- P2 pad 3: (no net) -> Net-(P2-Pad3)
- P2 pad 30: (no net) -> Net-(P2-Pad30)
- P2 pad 31: (no net) -> Net-(P2-Pad31)
- P2 pad 32: (no net) -> Net-(P2-Pad32)
- P2 pad 33: (no net) -> Net-(P2-Pad33)
- P2 pad 34: (no net) -> Net-(P2-Pad34)
- P2 pad 35: (no net) -> Net-(P2-Pad35)
- P2 pad 36: (no net) -> Net-(P2-Pad36)
- P2 pad 4: (no net) -> Net-(P2-Pad4)
- P2 pad 5: (no net) -> Net-(P2-Pad5)
- P2 pad 6: (no net) -> Net-(P2-Pad6)
- P2 pad 7: (no net) -> Net-(P2-Pad7)
- P2 pad 8: (no net) -> Net-(P2-Pad8)
- P2 pad 9: (no net) -> /CAN1_RX
Routing:
- added copper zone on F.Cu, net +3V3
- added copper zone on B.Cu, net GND
Other:
- board outline added: 63.5 x 119.4 mm
