File: LCC-CAN-Transceiver.sch (KiCad schematic (older format))
At the start: 18 parts, among them J201 Termination, J202 RJ45, J203 RJ45, T201 LCC Power Out, T202 LCC Power In, U201 LM358, U202 TCAN332DR

Commit message: Completed initial HW design.
Parts:
- C201: footprint Capacitors_THT:C_Rect_L4.0mm_W2.5mm_P2.50mm -> Capacitors_SMD:C_0603; Mouser Part Number 594-K104Z15Y5VF5TL2 -> 603-CC603KPX7R9BB104
- C202: footprint Capacitors_THT:C_Rect_L4.0mm_W2.5mm_P2.50mm -> Capacitors_SMD:C_0603; Mouser Part Number 594-K473K15X7RF5TL2 -> 963-GMK107BJ473KAHT
- C203: footprint Capacitors_THT:CP_Radial_D6.3mm_P2.50mm -> Capacitors_SMD:CP_Elec_4x5.8; Mouser Part Number 710-860080773002 -> 647-UUD1C150MCL
- D201: value CAN Tx -> LCC Tx; footprint LEDs:LED_D3.0mm -> LEDs:LED_0603; Mouser Part Number 710-151031SS04000 -> 710-150060SS75000
- D202: value CAN Rx -> LCC Rx; footprint LEDs:LED_D3.0mm -> LEDs:LED_0603; Mouser Part Number 710-151033YS03000 -> 710-150060YS75000
- D203, D204: footprint Diodes_THT:D_DO-15_P10.16mm_Horizontal -> Diodes_SMD:D_PowerDI-123; Mouser Part Number 625-SB240-E3/73 -> 621-DFLS240-7
- R201, R202: footprint Resistors_THT:R_Axial_DIN0204_L3.6mm_D1.6mm_P1.90mm_Vertical -> Resistors_SMD:R_0603; Mouser Part Number 603-CFR-25JB-52-160R -> 603-AC0603JR-07160RL
- R203, R204: footprint Resistors_THT:R_Axial_DIN0204_L3.6mm_D1.6mm_P2.54mm_Vertical -> Resistors_SMD:R_1206; Mouser Part Number 603-RSF2WSJT-52-60R -> 71-CRCW120660R0KNAIF
- U201: footprint Housings_DIP:DIP-8_W7.62mm -> Housings_SOIC:SOIC-8_3.9x4.9mm_Pitch1.27mm; Mouser Part Number 595-LM358AP -> 595-LM358DR
- U202: footprint Housings_SOIC:SOIC-8-1EP_3.9x4.9mm_Pitch1.27mm -> Housings_SOIC:SOIC-8_3.9x4.9mm_Pitch1.27mm
Changed lines of the file:
@@
 LIBS:lm2574n-5
 LIBS:sn65hvd233-ht
+LIBS:ap63205
 LIBS:LCC-PNET-Router-cache
 EELAYER 25 0
@@
 F 0 "U202" H 4600 2900 30  0000 C CNN
 F 1 "TCAN332DR" H 4600 3000 30  0000 C CNN
-F 2 "Housings_SOIC:SOIC-8-1EP_3.9x4.9mm_Pitch1.27mm" H 4600 2950 60  0001 C CNN
+F 2 "Housings_SOIC:SOIC-8_3.9x4.9mm_Pitch1.27mm" H 4600 2950 60  0001 C CNN
 F 3 "" H 4600 2950 60  0000 C CNN
 F 4 "595-TCAN332DR" H 4600 2950 60  0001 C CNN "Mouser Part Number"
@@
 NoConn ~ 4350 3150
 $Comp
-L +3.3V #PWR08
+L +3.3V #PWR203
 U 1 1 63C0330C
 P 4600 2450
-F 0 "#PWR08" H 4600 2300 50  0001 C CNN
+F 0 "#PWR203" H 4600 2300 50  0001 C CNN
 F 1 "+3.3V" H 4600 2590 50  0000 C CNN
 F 2 "" H 4600 2450 50  0001 C CNN
@@
 $EndComp
 $Comp
-L GND #PWR09
+L GND #PWR204
 U 1 1 63C0330D
 P 4600 3500
-F 0 "#PWR09" H 4600 3250 50  0001 C CNN
+F 0 "#PWR204" H 4600 3250 50  0001 C CNN
 F 1 "GND" H 4600 3350 50  0000 C CNN
 F 2 "" H 4600 3500 50  0001 C CNN
@@
 $EndComp
 $Comp
-L GND #PWR010
+L GND #PWR211
 U 1 1 63C0330E
 P 7400 3100
-F 0 "#PWR010" H 7400 2850 50  0001 C CNN
+F 0 "#PWR211" H 7400 2850 50  0001 C CNN
 F 1 "GND" H 7400 2950 50  0000 C CNN
 F 2 "" H 7400 3100 50  0001 C CNN
@@
 F 0 "C201" H 5275 2550 50  0000 L CNN
 F 1 ".1 uf" H 5275 2350 50  0000 L CNN
-F 2 "Capacitors_THT:C_Rect_L4.0mm_W2.5mm_P2.50mm" H 5288 2300 50  0001 C CNN
+F 2 "Capacitors_SMD:C_0603" H 5288 2300 50  0001 C CNN
 F 3 "" H 5250 2450 50  0001 C CNN
-F 4 "594-K104Z15Y5VF5TL2" H 5250 2450 60  0001 C CNN "Mouser Part Number"
+F 4 "603-CC603KPX7R9BB104" H 5250 2450 60  0001 C CNN "Mouser Part Number"
 	1    5250 2450
 	1    0    0    -1
@@
 F 0 "C203" H 5625 2550 50  0000 L CNN
 F 1 "15 uf 15V" H 5625 2350 50  0000 L CNN
-F 2 "Capacitors_THT:CP_Radial_D6.3mm_P2.50mm" H 5600 2450 50  0001 C CNN
+F 2 "Capacitors_SMD:CP_Elec_4x5.8" H 5600 2450 50  0001 C CNN
 F 3 "" H 5600 2450 50  0001 C CNN
-F 4 "710-860080773002" H 5600 2450 60  0001 C CNN "Mouser Part Number"
+F 4 "647-UUD1C150MCL" H 5600 2450 60  0001 C CNN "Mouser Part Number"
 	1    5600 2450
 	1    0    0    -1
@@
 F 0 "R203" V 5380 3400 50  0000 C CNN
 F 1 "60 Ohms" V 5300 3400 50  0000 C CNN
-F 2 "Resistors_THT:R_Axial_DIN0204_L3.6mm_D1.6mm_P2.54mm_Vertical" V 5230 3400 50  0001 C CNN
+F 2 "Resistors_SMD:R_1206" V 5230 3400 50  0001 C CNN
 F 3 "" H 5300 3400 50  0001 C CNN
-F 4 "603-RSF2WSJT-52-60R" V 5300 3400 60  0001 C CNN "Mouser Part Number"
+F 4 "71-CRCW120660R0KNAIF" V 5300 3400 60  0001 C CNN "Mouser Part Number"
 	1    5300 3400
 	1    0    0    -1
@@
 F 0 "R204" V 5880 3400 50  0000 C CNN
 F 1 "60 Ohms" V 5800 3400 50  0000 C CNN
-F 2 "Resistors_THT:R_Axial_DIN0204_L3.6mm_D1.6mm_P2.54mm_Vertical" V 5730 3400 50  0001 C CNN
+F 2 "Resistors_SMD:R_1206" V 5730 3400 50  0001 C CNN
 F 3 "" H 5800 3400 50  0001 C CNN
-F 4 "603-RSF2WSJT-52-60R" V 5800 3400 60  0001 C CNN "Mouser Part Number"
+F 4 "71-CRCW120660R0KNAIF" V 5800 3400 60  0001 C CNN "Mouser Part Number"
 	1    5800 3400
 	1    0    0    -1
@@
 F 0 "C202" H 5575 4450 50  0000 L CNN
 F 1 "47 nf" H 5575 4250 50  0000 L CNN
-F 2 "Capacitors_THT:C_Rect_L4.0mm_W2.5mm_P2.50mm" H 5588 4200 50  0001 C CNN
+F 2 "Capacitors_SMD:C_0603" H 5588 4200 50  0001 C CNN
 F 3 "" H 5550 4350 50  0001 C CNN
-F 4 "594-K473K15X7RF5TL2" H 5550 4350 60  0001 C CNN "Mouser Part Number"
+F 4 "963-GMK107BJ473KAHT" H 5550 4350 60  0001 C CNN "Mouser Part Number"
 	1    5550 4350
 	1    0    0    -1
 $EndComp
 $Comp
-L GND #PWR011
+L GND #PWR209
 U 1 1 63C03315
 P 5550 4750
-F 0 "#PWR011" H 5550 4500 50  0001 C CNN
+F 0 "#PWR209" H 5550 4500 50  0001 C CNN
 F 1 "GND" H 5550 4600 50  0000 C CNN
 F 2 "" H 5550 4750 50  0001 C CNN
@@
 $EndComp
 $Comp
-L +3.3V #PWR012
+L +3.3V #PWR208
 U 1 1 63C03316
 P 5450 2150
-F 0 "#PWR012" H 5450 2000 50  0001 C CNN
+F 0 "#PWR208" H 5450 2000 50  0001 C CNN
 F 1 "+3.3V" H 5450 2290 50  0000 C CNN
 F 2 "" H 5450 2150 50  0001 C CNN
@@
 $EndComp
 $Comp
-L GND #PWR013
+L GND #PWR207
 U 1 1 63C03317
 P 5400 2600
-F 0 "#PWR013" H 5400 2350 50  0001 C CNN
+F 0 "#PWR207" H 5400 2350 50  0001 C CNN
 F 1 "GND" H 5400 2450 50  0000 C CNN
 F 2 "" H 5400 2600 50  0001 C CNN
@@
 F 0 "D203" H 5900 1750 50  0000 C CNN
 F 1 "SB240" H 5900 1550 50  0000 C CNN
-F 2 "Diodes_THT:D_DO-15_P10.16mm_Horizontal" H 5900 1650 50  0001 C CNN
+F 2 "Diodes_SMD:D_PowerDI-123" H 5900 1650 50  0001 C CNN
 F 3 "" H 5900 1650 50  0001 C CNN
-F 4 "625-SB240-E3/73" H 5900 1650 60  0001 C CNN "Mouser Part Number"
+F 4 "621-DFLS240-7" H 5900 1650 60  0001 C CNN "Mouser Part Number"
 	1    5900 1650
 	1    0    0    -1
@@
 F 0 "D204" H 6650 1750 50  0000 C CNN
 F 1 "SB240" H 6650 1550 50  0000 C CNN
-F 2 "Diodes_THT:D_DO-15_P10.16mm_Horizontal" H 6650 1650 50  0001 C CNN
+F 2 "Diodes_SMD:D_PowerDI-123" H 6650 1650 50  0001 C CNN
 F 3 "" H 6650 1650 50  0001 C CNN
-F 4 "625-SB240-E3/73" H 6650 1650 60  0001 C CNN "Mouser Part Number"
+F 4 "621-DFLS240-7" H 6650 1650 60  0001 C CNN "Mouser Part Number"
 	1    6650 1650
 	1    0    0    -1
 $EndComp
 $Comp
-L GND #PWR014
+L GND #PWR210
 U 1 1 63C0331C
 P 6900 1800
-F 0 "#PWR014" H 6900 1550 50  0001 C CNN
+F 0 "#PWR210" H 6900 1550 50  0001 C CNN
 F 1 "GND" H 6900 1650 50  0000 C CNN
 F 2 "" H 6900 1800 50  0001 C CNN
@@
 F 0 "U201" H 3600 2150 50  0000 L CNN
 F 1 "LM358" H 3600 1750 50  0000 L CNN
-F 2 "Housings_DIP:DIP-8_W7.62mm" H 3600 1950 50  0001 C CNN
+F 2 "Housings_SOIC:SOIC-8_3.9x4.9mm_Pitch1.27mm" H 3600 1950 50  0001 C CNN
 F 3 "" H 3600 1950 50  0001 C CNN
-F 4 "595-LM358AP" H 3600 1950 60  0001 C CNN "Mouser Part Number"
+F 4 "595-LM358DR" H 3600 1950 60  0001 C CNN "Mouser Part Number"
 	2    3600 1950
 	1    0    0    1
@@
 F 0 "U201" H 3550 3600 50  0000 L CNN
 F 1 "LM358" H 3550 3200 50  0000 L CNN
-F 2 "Housings_DIP:DIP-8_W7.62mm" H 3550 3400 50  0001 C CNN
+F 2 "Housings_SOIC:SOIC-8_3.9x4.9mm_Pitch1.27mm" H 3550 3400 50  0001 C CNN
 F 3 "" H 3550 3400 50  0001 C CNN
-F 4 "595-LM358AP" H 3550 3400 60  0001 C CNN "Mouser Part Number"
+F 4 "595-LM358DR" H 3550 3400 60  0001 C CNN "Mouser Part Number"
 	1    3550 3400
 	1    0    0    -1
 $EndComp
 $Comp
-L GND #PWR015
+L GND #PWR202
 U 1 1 63C0331F
 P 3450 3800
-F 0 "#PWR015" H 3450 3550 50  0001 C CNN
+F 0 "#PWR202" H 3450 3550 50  0001 C CNN
 F 1 "GND" H 3450 3650 50  0000 C CNN
 F 2 "" H 3450 3800 50  0001 C CNN
@@
 $EndComp
 $Comp
-L +3.3V #PWR016
+L +3.3V #PWR201
 U 1 1 63C03320
 P 3450 3050
-F 0 "#PWR016" H 3450 2900 50  0001 C CNN
+F 0 "#PWR201" H 3450 2900 50  0001 C CNN
 F 1 "+3.3V" H 3450 3190 50  0000 C CNN
 F 2 "" H 3450 3050 50  0001 C CNN
@@
 F 0 "R201" H 4530 1500 50  0000 C CNN
 F 1 "160 Ohms" V 4450 1500 50  0000 C CNN
-F 2 "Resistors_THT:R_Axial_DIN0204_L3.6mm_D1.6mm_P1.90mm_Vertical" V 4380 1500 50  0001 C CNN
+F 2 "Resistors_SMD:R_0603" V 4380 1500 50  0001 C CNN
 F 3 "" H 4450 1500 50  0001 C CNN
-F 4 "603-CFR-25JB-52-160R" H 4450 1500 60  0001 C CNN "Mouser Part Number"
+F 4 "603-AC0603JR-07160RL" H 4450 1500 60  0001 C CNN "Mouser Part Number"
 	1    4450 1500
 	0    1    1    0
@@
 F 0 "R202" V 4580 3800 50  0000 C CNN
 F 1 "160 Ohms" V 4500 3800 50  0000 C CNN
-F 2 "Resistors_THT:R_Axial_DIN0204_L3.6mm_D1.6mm_P1.90mm_Vertical" V 4430 3800 50  0001 C CNN
+F 2 "Resistors_SMD:R_0603" V 4430 3800 50  0001 C CNN
 F 3 "" H 4500 3800 50  0001 C CNN
-F 4 "603-CFR-25JB-52-160R" V 4500 3800 60  0001 C CNN "Mouser Part Number"
+F 4 "603-AC0603JR-07160RL" V 4500 3800 60  0001 C CNN "Mouser Part Number"
 	1    4500 3800
 	0    1    1    0
@@
 P 4750 1250
 F 0 "D201" H 4750 1350 50  0000 C CNN
-F 1 "CAN Tx" H 4750 1150 50  0000 C CNN
-F 2 "LEDs:LED_D3.0mm" H 4750 1250 50  0001 C CNN
+F 1 "LCC Tx" H 4750 1150 50  0000 C CNN
+F 2 "LEDs:LED_0603" H 4750 1250 50  0001 C CNN
 F 3 "" H 4750 1250 50  0001 C CNN
-F 4 "710-151031SS04000" H 4750 1250 60  0001 C CNN "Mouser Part Number"
+F 4 "710-150060SS75000" H 4750 1250 60  0001 C CNN "Mouser Part Number"
 	1    4750 1250
 	0    -1   -1   0
@@
 P 4900 3600
 F 0 "D202" H 4900 3700 50  0000 C CNN
-F 1 "CAN Rx" H 4900 3500 50  0000 C CNN
-F 2 "LEDs:LED_D3.0mm" H 4900 3600 50  0001 C CNN
+F 1 "LCC Rx" H 4900 3500 50  0000 C CNN
+F 2 "LEDs:LED_0603" H 4900 3600 50  0001 C CNN
 F 3 "" H 4900 3600 50  0001 C CNN
-F 4 "710-151033YS03000" H 4900 3600 60  0001 C CNN "Mouser Part Number"
+F 4 "710-150060YS75000" H 4900 3600 60  0001 C CNN "Mouser Part Number"
 	1    4900 3600
 	0    -1   -1   0
@@
 	4900 3800 4650 3800
 $Comp
-L +3.3V #PWR017
+L +3.3V #PWR205
 U 1 1 63C03325
 P 4750 950
-F 0 "#PWR017" H 4750 800 50  0001 C CNN
+F 0 "#PWR205" H 4750 800 50  0001 C CNN
 F 1 "+3.3V" H 4750 1090 50  0000 C CNN
 F 2 "" H 4750 950 50  0001 C CNN
@@
 $EndComp
 $Comp
-L +3.3V #PWR018
+L +3.3V #PWR206
 U 1 1 63C03326
 P 4900 3350
-F 0 "#PWR018" H 4900 3200 50  0001 C CNN
+F 0 "#PWR206" H 4900 3200 50  0001 C CNN
 F 1 "+3.3V" H 4900 3490 50  0000 C CNN
 F 2 "" H 4900 3350 50  0001 C CNN
