File: LCC-PNET-Router.sch (KiCad schematic (older format))
At the start: 3 parts, among them J101 USB_A, P1 POCKETBEAGLE-P1, P2 POCKETBEAGLE-P2

Commit message: Finalize Parts Lists, generate Gerbers, etc.
Parts:
- P1, P2: Mouser Part Number (none) -> 517-929975-01-18-RK
Changed lines of the file:
@@
 F 2 "Socket_Strips:Socket_Strip_Straight_2x18_Pitch2.54mm" H 2850 2550 60  0001 C CNN
 F 3 "" H 2850 2550 60  0000 C CNN
+F 4 "517-929975-01-18-RK" H 2850 2550 60  0001 C CNN "Mouser Part Number"
 	1    2850 2550
 	1    0    0    -1
@@
 F 2 "Socket_Strips:Socket_Strip_Straight_2x18_Pitch2.54mm" H 5150 2550 60  0001 C CNN
 F 3 "" H 5150 2550 60  0000 C CNN
+F 4 "517-929975-01-18-RK" H 5150 2550 60  0001 C CNN "Mouser Part Number"
 	1    5150 2550
 	1    0    0    -1
