File: PowerSupply.sch (KiCad schematic (older format))
At the start: 6 parts, among them U401 AP63205

Commit message: Add Schematic PDF.
Connections:
- net +5V renamed 5V Out
Changed lines of the file:
@@
 $EndDescr
-$Comp
-L +5V #PWR029
-U 1 1 6411E143
-P 5600 4700
-F 0 "#PWR029" H 5600 4550 50  0001 C CNN
-F 1 "+5V" H 5600 4840 50  0000 C CNN
-F 2 "" H 5600 4700 50  0001 C CNN
-F 3 "" H 5600 4700 50  0001 C CNN
-	1    5600 4700
-	1    0    0    -1
-$EndComp
 $Comp
 L AP63205 U401
@@
 Text HLabel 3350 4600 0    60   Input ~ 0
 12-15 Volt input
+Text HLabel 5600 4700 2    60   Output ~ 0
+5V Out
 $EndSCHEMATC

Commit message: Finalize Parts Lists, generate Gerbers, etc.
Parts:
- C403, C404: Mouser Part Number 603-CC0603MRX6S5B226 -> 81-GRM188R60G226ME0J
Changed lines of the file:
@@
 F 2 "Capacitors_SMD:C_0603" H 5375 4875 50  0001 C CNN
 F 3 "" H 5375 4875 50  0001 C CNN
-F 4 "603-CC0603MRX6S5B226" H 5375 4875 60  0001 C CNN "Mouser Part Number"
+F 4 "81-GRM188R60G226ME0J" H 5375 4875 60  0001 C CNN "Mouser Part Number"
 	1    5375 4875
 	1    0    0    -1
@@
 F 2 "Capacitors_SMD:C_0603" H 5600 4875 50  0001 C CNN
 F 3 "" H 5600 4875 50  0001 C CNN
-F 4 "603-CC0603MRX6S5B226" H 5600 4875 60  0001 C CNN "Mouser Part Number"
+F 4 "81-GRM188R60G226ME0J" H 5600 4875 60  0001 C CNN "Mouser Part Number"
 	1    5600 4875
 	1    0    0    -1
